Commit message: adding galactic
adding galactic

File: amber_arm_moveit_config/srdf/amber_arm.srdf.xacro (robot description, xacro)
@@ -4,6 +4,6 @@
     A URDF file must exist for this robot as well, where the joints and the links that are referenced are defined
 -->
-<robot xmlns:xacro="http://www.ros.org/wiki/xacro" name="amberb1">
-  <xacro:include filename="$(find amber_moveit2_config)/srdf/amber_arm.xacro" />
-  <xacro:arm />
+<robot xmlns:xacro="http://www.ros.org/wiki/xacro" name="amber_arm">
+  <xacro:include filename="$(find amber_moveit_config)/srdf/amber_arm.xacro" />
+  <xacro:amber_arm />
 </robot>

File: amber_arm_moveit_config/srdf/amber_arm.xacro (robot description, xacro)
@@ -1,5 +1,5 @@
 <?xml version="1.0" ?>
-<robot xmlns:xacro="http://www.ros.org/wiki/xacro" name="amberb1">
-  <xacro:macro name="arm">
+<robot xmlns:xacro="http://www.ros.org/wiki/xacro" name="amber_arm">
+  <xacro:macro name="amber_arm">
     <!--GROUPS: Representation of a set of joints and links. This can be useful for specifying DOF to plan for, defining arms, end effectors, etc-->
     <!--LINKS: When a link is specified, the parent joint of that link (if it exists) is automatically included-->
@@ -19,5 +19,5 @@
     <!--END EFFECTOR: Purpose: Represent information about an end effector.-->
     <!--VIRTUAL JOINT: Purpose: this element defines a virtual joint between a robot link and an external frame of reference (considered fixed with respect to the robot)-->
-    <!-- <virtual_joint name="virtual_joint" type="floating" parent_frame="world" child_link="indy7_link0" /> -->
+    <virtual_joint name="fixed_frame" type="fixed" parent_frame="world" child_link="base_link">
     <!--DISABLE COLLISIONS: By default it is assumed that any link of the robot could potentially come into collision with any other link in the robot. This tag disables collision checking between a specified pair of links. -->
     <disable_collisions link1="base_link" link2="one_Link" reason="Adjacent"/>

File: amber_b1_description/urdf/amber_b1.ros2_control.xacro (robot description, xacro)
@@ -7,4 +7,7 @@
                 <param name="is_hw">${is_hw}</param>
                 <param name="is_ethercat">${is_ethercat}</param>
+            </hardware>
+            <hardware>
+                <plugin>fake_components/GenericSystem</plugin>
             </hardware>
             <joint name="${prefix}joint1">

File: amber_b1_description/urdf/amber_b1.urdf.xacro (robot description, xacro)
@@ -1,4 +1,4 @@
 <?xml version="1.0"?>
-<robot xmlns:xacro="http://www.ros.org/wiki/xacro" name="amber_b1">
+<robot xmlns:xacro="http://www.ros.org/wiki/xacro" name="amber_arm">
     <xacro:arg name="prefix" default="" />
     <xacro:arg name="is_hw" default="1"/>

File: amber_b1_description/urdf/amber_b1d.urdf (robot description, URDF)
Before this commit: robot None, 0 links, 0 joints
Links:
- added link base_link, mass 0.54367; collision mesh filename=file:///$(find amber_b1_description)/meshes/base_link.STL; visual mesh filename=file:///$(find amber_b1_description)/meshes/base_link.STL
- added link five_Link, mass 0.3436; collision mesh filename=file:///$(find amber_b1_description)/meshes/five_Link.STL; visual mesh filename=file:///$(find amber_b1_description)/meshes/five_Link.STL
- added link four_Link, mass 0.52945; collision mesh filename=file:///$(find amber_b1_description)/meshes/four_Link.STL; visual mesh filename=file:///$(find amber_b1_description)/meshes/four_Link.STL
- added link link_eef
- added link one_Link, mass 0.45633; collision mesh filename=file:///$(find amber_b1_description)/meshes/one_Link.STL; visual mesh filename=file:///$(find amber_b1_description)/meshes/one_Link.STL
- added link seven_Link, mass 0.046213; collision mesh filename=file:///$(find amber_b1_description)/meshes/seven_Link.STL; visual mesh filename=file:///$(find amber_b1_description)/meshes/seven_Link.STL
- added link six_Link, mass 0.47734; collision mesh filename=file:///$(find amber_b1_description)/meshes/six_Link.STL; visual mesh filename=file:///$(find amber_b1_description)/meshes/six_Link.STL
- added link three_Link, mass 0.45615; collision mesh filename=file:///$(find amber_b1_description)/meshes/three_Link.STL; visual mesh filename=file:///$(find amber_b1_description)/meshes/three_Link.STL
- added link two_Link, mass 0.66129; collision mesh filename=file:///$(find amber_b1_description)/meshes/two_Link.STL; visual mesh filename=file:///$(find amber_b1_description)/meshes/two_Link.STL
- added link world
Joints:
- added joint amber_joint_base: type fixed, parent world, child base_link, origin xyz=0 0 0 rpy=0 0 0
- added joint joint1: type revolute, parent base_link, child one_Link, origin xyz=0 0 0.0825 rpy=0 0 0, axis 0 0 1, limit lower=-2.4435 upper=2.4435 effort=100 velocity=3.1415
- added joint joint2: type revolute, parent one_Link, child two_Link, origin xyz=0 0.0275 0.0853 rpy=-1.5708 0 0, axis 0 0 1, limit lower=-2.3213 upper=2.3213 effort=100 velocity=3.1415
- added joint joint3: type revolute, parent two_Link, child three_Link, origin xyz=0 -0.1289 -0.0275 rpy=1.5708 0 0, axis 0 0 1, limit lower=-2.2863 upper=2.2863 effort=100 velocity=3.1415
- added joint joint4: type revolute, parent three_Link, child four_Link, origin xyz=0 -0.0275 0.0853 rpy=-1.5708 0 0, axis 0 0 1, limit lower=-2.2863 upper=2.2863 effort=100 velocity=3.1415
- added joint joint5: type revolute, parent four_Link, child five_Link, origin xyz=0 -0.1251 0.0275 rpy=1.5708 0 0, axis 0 0 1, limit lower=-2.2863 upper=2.2863 effort=100 velocity=5.23
- added joint joint6: type revolute, parent five_Link, child six_Link, origin xyz=0 0.0251 0.079 rpy=-1.5708 0 0, axis 0 0 1, limit lower=-2.2863 upper=2.2863 effort=100 velocity=5.23
- added joint joint7: type revolute, parent six_Link, child seven_Link, origin xyz=0 -0.1236 -0.0251 rpy=1.5708 0 0, axis 0 0 1, limit lower=-3.05 upper=3.05 effort=100 velocity=5.23
- added joint joint_eef: type fixed, parent seven_Link, child link_eef, origin xyz=0 0 0.0385 rpy=0 0 0
