Commit message: adding files
adding files

File: amber_b1_description/urdf/amber_b1.ros2_control.xacro (robot description, xacro)
@@ -11,5 +11,5 @@
                 <plugin>fake_components/GenericSystem</plugin>
             </hardware>
-            <joint name="${prefix}joint1">
+            <joint name="joint1">
                 <command_interface name="position">
                     <param name="min">-2.4435</param>
@@ -24,5 +24,5 @@
                 <state_interface name="effort"/>
             </joint>
-            <joint name="${prefix}joint2">
+            <joint name="joint2">
                 <command_interface name="position">
                     <param name="min">-2.3213</param>
@@ -37,5 +37,5 @@
                 <state_interface name="effort"/>
             </joint>
-            <joint name="${prefix}joint3">
+            <joint name="joint3">
                 <command_interface name="position">
                     <param name="min">-2.2863</param>
@@ -50,5 +50,5 @@
                 <state_interface name="effort"/>
             </joint>
-            <joint name="${prefix}joint4">
+            <joint name="joint4">
                 <command_interface name="position">
                     <param name="min">-2.2863</param>
@@ -63,5 +63,5 @@
                 <state_interface name="effort"/>
             </joint>
-            <joint name="${prefix}joint5">
+            <joint name="joint5">
                 <command_interface name="position">
                     <param name="min">-2.2863</param>
@@ -76,5 +76,5 @@
                 <state_interface name="effort"/>
             </joint>
-            <joint name="${prefix}joint6">
+            <joint name="joint6">
                 <command_interface name="position">
                     <param name="min">-2.2863</param>
@@ -89,5 +89,5 @@
                 <state_interface name="effort"/>
             </joint>
-            <joint name="${prefix}joint7">
+            <joint name="joint7">
                 <command_interface name="position">
                     <param name="min">-3.05</param>

File: amber_b1_description/urdf/amber_b1.urdf.xacro (robot description, xacro)
@@ -6,5 +6,5 @@
     <xacro:include filename="$(find amber_b1_description)/urdf/amber_b1_description.urdf.xacro" />
     <xacro:include filename="$(find amber_b1_description)/urdf/amber_b1.ros2_control.xacro" />
-    <xacro:amberb1 prefix="$(arg prefix)"/>
+    <xacro:amber_arm prefix="$(arg prefix)"/>
     <xacro:amberb1_ros2_control prefix="$(arg prefix)" is_hw="$(arg is_hw)" is_ethercat="$(arg is_ethercat)"/>
 </robot>

File: amber_b1_description/urdf/amber_b1_description.urdf.xacro (robot description, xacro)
@@ -1,5 +1,5 @@
 <?xml version="1.0"?>
 <robot xmlns:xacro="http://www.ros.org/wiki/xacro">
-    <xacro:macro name="amberb1" params="prefix">
+    <xacro:macro name="amber_arm" params="prefix">
     <material name="${prefix}Silver">
         <color rgba="0.753 0.753 0.753 1.0"/>

Commit message: Update amber_b1.ros2_control.xacro

File: amber_b1_description/urdf/amber_b1.ros2_control.xacro (robot description, xacro)
@@ -1,6 +1,6 @@
 <?xml version="1.0"?>
 <robot xmlns:xacro="http://ros.org/wiki/xacro">
-    <xacro:macro name="amberb1_ros2_control" params="prefix is_hw is_ethercat">
-        <ros2_control name="amber_b1_position" type="system">
+    <xacro:macro name="amber_arm" params="prefix is_hw is_ethercat">
+        <ros2_control name="amber_arm" type="system">
             <hardware>
                 <plugin>AmberB1Hardware</plugin>
@@ -8,7 +8,14 @@
                 <param name="is_ethercat">${is_ethercat}</param>
             </hardware>
-            <hardware>
+        <xacro:if value="${gazebo}">
+         <hardware>
+            <plugin>gazebo_ros2_control/GazeboSystem</plugin>
+         </hardware>
+        </xacro:if>
+        <xacro:unless value="${gazebo}">
+             <hardware>
                 <plugin>fake_components/GenericSystem</plugin>
             </hardware>
+        </xacro:unless>
             <joint name="joint1">
                 <command_interface name="position">
@@ -103,4 +110,11 @@
             </joint>
         </ros2_control>
+        <gazebo>
+            <plugin filename="libgazebo_ros2_control.so" name="gazebo_ros2_control_urdf">
+                <robot_param>robot_description</robot_param>
+                <robot_param_node>robot_state_publisher</robot_param_node>
+                <parameters>$(find amber_arm_moveit_config)/config/ros_controllers.yaml</parameters>
+            </plugin>
+        </gazebo>
     </xacro:macro>
 </robot>

Commit message: edit

File: amber_b1_description/urdf/amber_b1.ros2_control.xacro (robot description, xacro)
@@ -1,21 +1,20 @@
-<?xml version="1.0"?>
+<?xml version="1.0" encoding="UTF-8"?>
 <robot xmlns:xacro="http://ros.org/wiki/xacro">
-    <xacro:macro name="amber_arm" params="prefix is_hw is_ethercat">
-        <ros2_control name="amber_arm" type="system">
-                <xacro:if value="${gazebo}">
-            <hardware>
-                <plugin>gazebo_ros2_control/GazeboSystem</plugin>
-            </hardware>
-            <hardware>
+   <ros2_control name="amber_arm_control" type="system">
+      <xacro:if value="${gazebo}">
+         <hardware>
+            <plugin>gazebo_ros2_control/GazeboSystem</plugin>
+         </hardware>
+      </xacro:if>
+      <xacro:unless value="${gazebo}">
+         <hardware>
+            <plugin>fake_components/GenericSystem</plugin>
+         </hardware>
+      </xacro:unless>
+        <hardware>
                 <plugin>AmberB1Hardware</plugin>
                 <param name="is_hw">${is_hw}</param>
                 <param name="is_ethercat">${is_ethercat}</param>
-            </hardware>
-                </xacro:if>
-                <xacro:unless value="${gazebo}">
-             <hardware>
-                        <plugin>fake_components/GenericSystem</plugin>
-            </hardware>
-                </xacro:unless>
+        </hardware>
             <joint name="joint1">
                 <command_interface name="position">

File: amber_b1_description/urdf/amber_b1.urdf.xacro (robot description, xacro)
@@ -1,10 +1,14 @@
 <?xml version="1.0"?>
 <robot xmlns:xacro="http://www.ros.org/wiki/xacro" name="amber_arm">
-    <xacro:arg name="prefix" default="" />
-    <xacro:arg name="is_hw" default="1"/>
-    <xacro:arg name="is_ethercat" default="0"/>
-    <xacro:include filename="$(find amber_b1_description)/urdf/amber_b1_description.urdf.xacro" />
-    <xacro:include filename="$(find amber_b1_description)/urdf/amber_b1.ros2_control.xacro" />
-    <xacro:amber_arm prefix="$(arg prefix)"/>
-    <xacro:amberb1_ros2_control prefix="$(arg prefix)" is_hw="$(arg is_hw)" is_ethercat="$(arg is_ethercat)"/>
+	<xacro:macro name="amber_arm" params="use_sim_time">
+		<xacro:property name="gazebo" value="${use_sim_time}" />
+    		<xacro:arg name="prefix" default="" />
+    		<xacro:arg name="is_hw" default="1"/>
+    		<xacro:arg name="is_ethercat" default="0"/>
+    		<xacro:arg name="use_sim_time" default="false" />
+    		<xacro:include filename="$(find amber_b1_description)/urdf/amber_b1_description.urdf.xacro" />
+    		<xacro:include filename="$(find amber_b1_description)/urdf/amber_b1.ros2_control.xacro" />
+    		<xacro:amber_arm prefix="$(arg prefix)"/>
+    		<xacro:amber_arm_control prefix="$(arg prefix)" is_hw="$(arg is_hw)" is_ethercat="$(arg is_ethercat)"/>
+    	</xacro:macro>
 </robot>
